File: eda/vectorscope.kicad_pcb (KiCad board)
At the start: 2 copper layers, 116 x 73 mm, 121 parts, among them M1 PICO, SW1 tactile key, SW10 Comment, SW11 Comment, SW12 Comment, SW13 Comment, SW2 tactile key, SW3 tactile key, SW4 tactile key, SW5 tactile key, SW6 tactile key, SW7 tactile key, SW8 tactile key, SW9 tactile key, T1 DMN65D8L-7, U1 AK4619, U2 LMV324, U3 TLC59283, U4 TPA321

Commit message: fixed typo in footprint library name (missing dot, .vector-orig)
Parts:
- ? (x59): footprint vector-orig: -> .vector-orig:
- C1, C2: footprint vector-orig:_Users_Voja_Desktop_Projekti_Gio.PcbLib_Tantal -> .vector-orig:_Users_Voja_Desktop_Projekti_Gio.PcbLib_Tantal
- C10, C11, C12, C13, C14, C15, C16, C17, C18, C19, C20, C3, C4, C5, C6, C7, C8, C9, R1, R10, R11, R12, R13, R2, R3, R4, R5, R6, R7, R8, R9: footprint vector-orig:_Users_Voja_Desktop_CUBE_ESP.PcbLib_TANTALUM KEMET C -> .vector-orig:_Users_Voja_Desktop_CUBE_ESP.PcbLib_TANTALUM KEMET C
- L1: footprint vector-orig:0805 -> .vector-orig:0805
- LY1, LY2, LY3, LY4, LY5, LY6, LY7, LY8: footprint vector-orig:_Users_Voja_Desktop_ESP.PcbLib_LED0603 -> .vector-orig:_Users_Voja_Desktop_ESP.PcbLib_LED0603
- M1: footprint vector-orig:_Users_Voja_Desktop_Projekti_Gio.PcbLib_PICO -> .vector-orig:_Users_Voja_Desktop_Projekti_Gio.PcbLib_PICO
- SW1, SW2, SW3, SW4, SW5, SW6, SW7, SW8, SW9: footprint vector-orig:_Users_Voja_Documents_GitHub_willo-pcb_ESP.PcbLib_key4p -> .vector-orig:_Users_Voja_Documents_GitHub_willo-pcb_ESP.PcbLib_key4p
- SW10, SW11, SW12: footprint vector-orig:key 12x12 SMD -> .vector-orig:key 12x12 SMD
- SW13: footprint vector-orig:_Users_Voja_Desktop_Projekti_Gio.PcbLib_JOYSTICK 2 -> .vector-orig:_Users_Voja_Desktop_Projekti_Gio.PcbLib_JOYSTICK 2
- T1, ZD1: footprint vector-orig:SOT-23 -> .vector-orig:SOT-23
- U1: footprint vector-orig:AK4619 -> .vector-orig:AK4619
- U2: footprint vector-orig:TSSOP 14 -> .vector-orig:TSSOP 14
- U3: footprint vector-orig:_Users_Voja_Desktop_Projekti_Gio.PcbLib_TQFN24 -> .vector-orig:_Users_Voja_Desktop_Projekti_Gio.PcbLib_TQFN24
- U4: footprint vector-orig:_Users_Voja_Desktop_CUBE_ESP.PcbLib_MSOP8 -> .vector-orig:_Users_Voja_Desktop_CUBE_ESP.PcbLib_MSOP8
